Commit message: new_urdf_structure

File: my-robot/robot.urdf (robot description, URDF)
Before this commit: robot my-robot, 2 links, 1 joints
Links:
- removed link base_robot
- removed link shaft_base
- added link part_1, mass 0.51392; collision mesh filename=assets/part_1.stl; visual mesh filename=assets/part_1.stl
Joints:
- removed joint 1revolute

Commit message: A_Robot_in_Urdf

File: my-robot/robot.urdf (robot description, URDF)
Before this commit: robot D:\python_projects\onshape_urdf\my-robot, 1 links, 0 joints
Links:
- removed link part_1
- added link base_link, mass 1.0; collision mesh filename=assets/part_1.stl; visual mesh filename=assets/part_1.stl
